File: small/_autosave-saxli.kicad_pcb (KiCad board)
At the start: 4 copper layers, 157.7 x 103.4 mm, 147 parts, among them IC1 PIC32MX350F256H-V_PT, J10 Conn_01x06_Female, J2 Screw_Terminal_01x02, J3 Micro_SD_Card, J4 Conn_01x05_Female, J5 Conn_02x04_Odd_Even, J6 RJ45_Amphenol_RJMG1BD3B8K1ANR, J7 Screw_Terminal_01x08, J8 Screw_Terminal_01x08, J9 Screw_Terminal_01x08, Q1 2N7002, U1 LM358, U10 TPS5430DDAR, U11 EL357N(C)(TA)-G, U12 EL357N(C)(TA)-G, U13 ASSR-1218, U14 SIM800C, U15 ASSR-1218, U16 SRV05-4, U18 ULN2003A, U2 LM7805_TO220, U20 TPS5430DDAR, U3 LD1117S33TR_SOT223, U4 ENC28J60x-SS, U5 AT25M02, U6 EL357N(C)(TA)-G, U7 EL357N(C)(TA)-G, U8 PCF8563T, U9 ISO1540, Y1 Crystal, Y2 Crystal

Commit message: sim800 changed to sim808
Parts:
- moved U14 2.80 mm to (167.3, 42.8)
Changed lines of the file:
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@@
   )
   (module RF_GSM:SIMCom_SIM800C (layer F.Cu)
-    (at 165.088 44.572)
+    (at 167.259 42.799)
     (descr "Quad-Band GSM/GPRS module, 17.6x15.7x2.3mm, http://simcom.ee/documents/SIM800C/SIM800C_Hardware_Design_V1.05.pdf")
     (tags "GSM Module SIM800C")
