File: small/ethernet.sch (KiCad schematic (older format))
At the start: 26 parts, among them J6 RJ45_Amphenol_RJMG1BD3B8K1ANR, U4 ENC28J60x-SS, Y1 Crystal

Commit message: ENC28j60 package changed to soic 28 17.9
TODO: route
Parts:
- J6: LCSC (none) -> N/A
- R22, R23: LCSC C7250 -> C7250
- U4: footprint Package_SO:SSOP-28_5.3x10.2mm_P0.65mm -> Package_SO:SOIC-28W_7.5x17.9mm_P1.27mm; Price (none) -> 3.2879
Changed lines of the file:
@@
 F 0 "U4" H 3350 3000 50  0000 C CNN
 F 1 "ENC28J60x-SS" H 3325 3200 50  0000 C CNN
-F 2 "Package_SO:SSOP-28_5.3x10.2mm_P0.65mm" H 4500 2050 50  0001 C CIN
+F 2 "Package_SO:SOIC-28W_7.5x17.9mm_P1.27mm" H 4500 2050 50  0001 C CIN
 F 3 "http://ww1.microchip.com/downloads/en/devicedoc/39662e.pdf" H 3350 3000 50  0001 C CNN
 F 4 " C47351" H 3350 3000 50  0001 C CNN "LCSC"
 F 5 "1" H 3350 3000 50  0001 C CNN "source"
+F 6 "3.2879" H 3350 3000 50  0001 C CNN "Price"
 	1    3350 3000
 	1    0    0    -1
@@
 F 2 "Resistor_SMD:R_0603_1608Metric" V 6580 2450 50  0001 C CNN
 F 3 "https://datasheet.lcsc.com/szlcsc/Uniroyal-Elec-0603WAF1005T5E_C7250.pdf" H 6650 2450 50  0001 C CNN
-F 4 " C7250" H 6650 2450 50  0001 C CNN "LCSC"
+F 4 "C7250" H 6650 2450 50  0001 C CNN "LCSC"
 F 5 "0.0028" H 6650 2450 50  0001 C CNN "Price"
 F 6 "0603WAF1005T5E" H 6650 2450 50  0001 C CNN "MPN"
@@
 F 2 "Connector_RJ:RJ45_Amphenol_RJMG1BD3B8K1ANR" H 7775 2175 50  0001 C CNN
 F 3 "https://www.amphenolcanada.com/ProductSearch/Drawings/AC/RJMG1BD3B8K1ANR.PDF" H 7775 2275 50  0001 C CNN
+F 4 "N/A" H 7775 1475 50  0001 C CNN "LCSC"
 	1    7775 1475
 	1    0    0    -1
@@
 F 2 "Resistor_SMD:R_0603_1608Metric" V 6805 2450 50  0001 C CNN
 F 3 "https://datasheet.lcsc.com/szlcsc/Uniroyal-Elec-0603WAF1005T5E_C7250.pdf" H 6875 2450 50  0001 C CNN
-F 4 " C7250" H 6875 2450 50  0001 C CNN "LCSC"
+F 4 "C7250" H 6875 2450 50  0001 C CNN "LCSC"
 F 5 "0.0028" H 6875 2450 50  0001 C CNN "Price"
 F 6 "0603WAF1005T5E" H 6875 2450 50  0001 C CNN "MPN"

Commit message: SPI change:
ENC28j60 on one spi
SDCARD and EEPROM on the other.
Parts:
- R4: value 2k 1% -> 2.32k 1%
Changed lines of the file:
@@
 AR Path="/60757620/607819FB" Ref="R4"  Part="1"
 F 0 "R4" V 4293 3600 50  0000 C CNN
-F 1 "2k 1%" V 4384 3600 50  0000 C CNN
+F 1 "2.32k 1%" V 4384 3600 50  0000 C CNN
 F 2 "Resistor_SMD:R_0603_1608Metric" V 4430 3600 50  0001 C CNN
 F 3 "https://datasheet.lcsc.com/szlcsc/Uniroyal-Elec-0603WAF2321T5E_C22905.pdf" H 4500 3600 50  0001 C CNN

Commit message: sdcard and clock capacitor added.
Changed lines of the file:
@@
 Text Label 6250 1975 0    50   ~ 0
 TPIN+
-Text Label 6425 975  0    50   ~ 0
+Text Label 6450 1175 0    50   ~ 0
 TPOUT-
-Text Label 6425 1175 0    50   ~ 0
+Text Label 6450 975  0    50   ~ 0
 TPOUT+
 Wire Wire Line
