File: small/power.sch (KiCad schematic (older format))
At the start: 28 parts, among them J2 Screw_Terminal_01x02, U10 TPS5430DDAR, U2 LM7805_TO220, U20 TPS5430DDAR, U3 LD1117S33TR_SOT223

Commit message: simcard colder changed to 78800-0001
Parts:
- D7, D9: LCSC (none) -> C8678
Changed lines of the file:
@@
 F 10 "" H 6000 3600 50  0001 L CNN "Arrow Part Number"
 F 11 "" H 6000 3500 50  0001 L CNN "Arrow Price/Stock"
+F 12 "C8678" H 5500 4250 50  0001 C CNN "LCSC"
 	1    5500 4250
 	0    1    1    0
@@
 F 10 "" H 6125 1825 50  0001 L CNN "Arrow Part Number"
 F 11 "" H 6125 1725 50  0001 L CNN "Arrow Price/Stock"
+F 12 "C8678" H 5625 2475 50  0001 C CNN "LCSC"
 	1    5625 2475
 	0    1    1    0

Commit message: BOM updated
Layout changed
Parts:
- C1, C2, C3, C32, C33, C34, C36, C37, C4, C42, U10, U20: source (none) -> 0
- C35, C40, C41, L1, L2: source (none) -> 1
- D3: MPN (none) -> FC-2012HRK-620D; Price (none) -> 0.0199; source (none) -> 0
- D7, D9: MPN (none) -> SS34B-HF; Manufacturer_Name Comchip Technology -> (none); Manufacturer_Part_Number SS34B-HF -> (none); Price (none) -> 0.0350; source (none) -> 0
- R27, R28: MPN (none) -> 0603WAF1002T5E; source (none) -> 0
- R31: MPN (none) -> 0603WAF1000T5E; source (none) -> 0
- R57: Price (none) -> 0.0016; source (none) -> 0
- R59: MPN (none) -> 0603WAF1101T5E; source (none) -> 0
- U2: MPN (none) -> CJ7805; Mpn CJ7805 -> (none); Website mouser -> (none); source (none) -> 1
- U3: MPN (none) -> LD1117S33CTR; Mpn LD1117S33CTR -> (none); Website mouser -> (none); source (none) -> 1
Changed lines of the file:
@@
 F 5 "0.7338" H 3900 2775 50  0001 C CNN "Price"
 F 6 "TPS5430DDAR" H 3900 2775 50  0001 C CNN "MPN"
+F 7 "0" H 3900 2775 50  0001 C CNN "source"
 	1    3900 2775
 	1    0    0    -1
@@
 F 4 "C13585" H 2825 2750 50  0001 C CNN "LCSC"
 F 5 "CL31A106KBHNNNE" H 2825 2750 50  0001 C CNN "MPN"
+F 6 "0" H 2825 2750 50  0001 C CNN "source"
 	1    2825 2750
 	1    0    0    -1
@@
 F 4 "C22764" H 7275 3300 50  0001 C CNN "LCSC"
 F 5 "0.0020" H 7275 3300 50  0001 C CNN "Price"
+F 6 "0603WAF1101T5E" H 7275 3300 50  0001 C CNN "MPN"
+F 7 "0" H 7275 3300 50  0001 C CNN "source"
 	1    7275 3300
 	1    0    0    -1
@@
 F 5 "0.1927" H 6125 4350 50  0001 C CNN "Price"
 F 6 "SLO1040H220MTT" H 6125 4350 50  0001 C CNN "MPN"
+F 7 "1" H 6125 4350 50  0001 C CNN "source"
 	1    6125 4350
 	1    0    0    -1
@@
 F 4 "C22994" H 7250 5075 50  0001 C CNN "LCSC"
 F 5 "0603WAF3241T5E" H 7250 5075 50  0001 C CNN "MPN"
+F 6 "0.0016" H 7250 5075 50  0001 C CNN "Price"
+F 7 "0" H 7250 5075 50  0001 C CNN "source"
 	1    7250 5075
 	1    0    0    -1
@@
 F 2 "Package_TO_SOT_SMD:SOT-223" H 5575 1125 50  0001 C CNN
 F 3 "https://datasheet.lcsc.com/szlcsc/STMicroelectronics-LD1117S33CTR_C35879.pdf" H 5675 675 50  0001 C CNN
-F 4 "LD1117S33CTR" H 5575 925 50  0001 C CNN "Mpn"
+F 4 "" H 5575 925 50  0001 C CNN "Mpn"
 F 5 "0.1762" H 5575 925 50  0001 C CNN "Price"
-F 6 "mouser" H 5575 925 50  0001 C CNN "Website"
+F 6 "" H 5575 925 50  0001 C CNN "Website"
 F 7 "C35879" H 5575 925 50  0001 C CNN "LCSC"
+F 8 "LD1117S33CTR" H 5575 925 50  0001 C CNN "MPN"
+F 9 "1" H 5575 925 50  0001 C CNN "source"
 	1    5575 925
 	1    0    0    -1
@@
 F 2 "Package_TO_SOT_SMD:TO-252-2" H 3675 1150 50  0001 C CIN
 F 3 "https://datasheet.lcsc.com/szlcsc/Changjiang-Electronics-Tech-CJ-CJ7805-3_C21706.pdf" H 3675 875 50  0001 C CNN
-F 4 "CJ7805" H 3675 925 50  0001 C CNN "Mpn"
+F 4 "" H 3675 925 50  0001 C CNN "Mpn"
 F 5 "0.1620" H 3675 925 50  0001 C CNN "Price"
-F 6 "mouser" H 3675 925 50  0001 C CNN "Website"
+F 6 "" H 3675 925 50  0001 C CNN "Website"
 F 7 "C21706" H 3675 925 50  0001 C CNN "LCSC"
+F 8 "CJ7805" H 3675 925 50  0001 C CNN "MPN"
+F 9 "1" H 3675 925 50  0001 C CNN "source"
 	1    3675 925
 	1    0    0    -1
@@
 F 5 "0.0195" H 3075 1050 50  0001 C CNN "Price"
 F 6 "CL21B105KBFNNNE" H 3075 1050 50  0001 C CNN "MPN"
+F 7 "0" H 3075 1050 50  0001 C CNN "source"
 	1    3075 1050
 	1    0    0    -1
@@
 F 5 "0.0071" H 4175 1075 50  0001 C CNN "Price"
 F 6 "CC0603KRX7R9BB104" H 4175 1075 50  0001 C CNN "MPN"
+F 7 "0" H 4175 1075 50  0001 C CNN "source"
 	1    4175 1075
 	1    0    0    -1
@@
 F 5 "0.0071" H 4925 1075 50  0001 C CNN "Price"
 F 6 "CC0603KRX7R9BB104" H 4925 1075 50  0001 C CNN "MPN"
+F 7 "0" H 4925 1075 50  0001 C CNN "source"
 	1    4925 1075
 	1    0    0    -1
@@
 F 5 "VEH221M1VTR" H 6775 2850 50  0001 C CNN "MPN"
 F 6 "0.1259" H 6775 2850 50  0001 C CNN "Price"
+F 7 "1" H 6775 2850 50  0001 C CNN "source"
 	1    6775 2850
 	1    0    0    -1
@@
 F 5 "VEH221M1VTR" H 6750 4625 50  0001 C CNN "MPN"
 F 6 "0.1259" H 6750 4625 50  0001 C CNN "Price"
+F 7 "1" H 6750 4625 50  0001 C CNN "source"
 	1    6750 4625
 	1    0    0    -1
@@
 F 5 "VEH221M1VTR" H 6450 1075 50  0001 C CNN "MPN"
 F 6 "0.1259" H 6450 1075 50  0001 C CNN "Price"
+F 7 "1" H 6450 1075 50  0001 C CNN "source"
 	1    6450 1075
 	1    0    0    -1
@@
 F 5 "TAJA106K016RNJ" H 6850 1075 50  0001 C CNN "MPN"
 F 6 "0.2135" H 6850 1075 50  0001 C CNN "Price"
+F 7 "0" H 6850 1075 50  0001 C CNN "source"
 	1    6850 1075
 	1    0    0    -1
@@
 F 5 "0.0053" H 4750 4350 50  0001 C CNN "Price"
 F 6 "0603B103K500NT" H 4750 4350 50  0001 C CNN "MPN"
+F 7 "0" H 4750 4350 50  0001 C CNN "source"
 	1    4750 4350
 	0    -1   -1   0
@@
 F 4 "C13585" H 2800 4525 50  0001 C CNN "LCSC"
 F 5 "CL31A106KBHNNNE" H 2800 4525 50  0001 C CNN "MPN"
+F 6 "0" H 2800 4525 50  0001 C CNN "source"
 	1    2800 4525
 	1    0    0    -1
@@
 F 5 "0.1927" H 6150 2575 50  0001 C CNN "Price"
 F 6 "SLO1040H220MTT" H 6150 2575 50  0001 C CNN "MPN"
+F 7 "1" H 6150 2575 50  0001 C CNN "source"
 	1    6150 2575
 	1    0    0    -1
@@
 F 5 "0.7338" H 3875 4550 50  0001 C CNN "Price"
 F 6 "TPS5430DDAR" H 3875 4550 50  0001 C CNN "MPN"
+F 7 "0" H 3875 4550 50  0001 C CNN "source"
 	1    3875 4550
 	1    0    0    -1
@@
 F 5 "TAJA106K016RNJ" H 6500 2725 50  0001 C CNN "MPN"
 F 6 "0.2135" H 6500 2725 50  0001 C CNN "Price"
+F 7 "0" H 6500 2725 50  0001 C CNN "source"
 	1    6500 2725
 	1    0    0    -1
@@
 F 5 "TAJA106K016RNJ" H 6475 4500 50  0001 C CNN "MPN"
 F 6 "0.2135" H 6475 4500 50  0001 C CNN "Price"
+F 7 "0" H 6475 4500 50  0001 C CNN "source"
 	1    6475 4500
 	1    0    0    -1
@@
 F 4 "C25804" H 7275 2825 50  0001 C CNN "LCSC"
 F 5 "0.02" H 7275 2825 50  0001 C CNN "Price"
+F 6 "0603WAF1002T5E" H 7275 2825 50  0001 C CNN "MPN"
+F 7 "0" H 7275 2825 50  0001 C CNN "source"
 	1    7275 2825
 	1    0    0    -1
@@
 F 4 "C25804" H 7250 4600 50  0001 C CNN "LCSC"
 F 5 "0.02" H 7250 4600 50  0001 C CNN "Price"
+F 6 "0603WAF1002T5E" H 7250 4600 50  0001 C CNN "MPN"
+F 7 "0" H 7250 4600 50  0001 C CNN "source"
 	1    7250 4600
 	1    0    0    -1
@@
 F 4 "C22775" H 7075 1450 50  0001 C CNN "LCSC"
 F 5 "0.0019" H 7075 1450 50  0001 C CNN "Price"
+F 6 "0603WAF1000T5E" H 7075 1450 50  0001 C CNN "MPN"
+F 7 "0" H 7075 1450 50  0001 C CNN "source"
 	1    7075 1450
 	1    0    0    -1
@@
 F 3 "https://datasheet.lcsc.com/szlcsc/Foshan-NationStar-Optoelectronics-FC-2012HRK-620D_C84256.pdf" H 7075 1150 50  0001 C CNN
 F 4 "C84256" V 7075 1150 50  0001 C CNN "LCSC"
+F 5 "FC-2012HRK-620D" H 7075 1150 50  0001 C CNN "MPN"
+F 6 "0.0199" H 7075 1150 50  0001 C CNN "Price"
+F 7 "0" H 7075 1150 50  0001 C CNN "source"
 	1    7075 1150
 	0    -1   -1   0
@@
 F 5 "0.0053" H 4775 2575 50  0001 C CNN "Price"
 F 6 "0603B103K500NT" H 4775 2575 50  0001 C CNN "MPN"
+F 7 "0" H 4775 2575 50  0001 C CNN "source"
 	1    4775 2575
 	0    -1   -1   0
@@
 F 4 "Schottky Diodes & Rectifiers DIODE SCHOTTKY 3A 40V SMB" H 6000 4200 50  0001 L CNN "Description"
 F 5 "3.2" H 6000 4100 50  0001 L CNN "Height"
-F 6 "Comchip Technology" H 6000 4000 50  0001 L CNN "Manufacturer_Name"
-F 7 "SS34B-HF" H 6000 3900 50  0001 L CNN "Manufacturer_Part_Number"
+F 6 "" H 6000 4000 50  0001 L CNN "Manufacturer_Name"
+F 7 "" H 6000 3900 50  0001 L CNN "Manufacturer_Part_Number"
 F 8 "750-SS34B-HF" H 6000 3800 50  0001 L CNN "Mouser Part Number"
 F 9 "https://www.mouser.co.uk/ProductDetail/Comchip-Technology/SS34B-HF/?qs=vmHwEFxEFR9G1M%252BcUPG%2FxQ%3D%3D" H 6000 3700 50  0001 L CNN "Mouser Price/Stock"
@@
 F 11 "" H 6000 3500 50  0001 L CNN "Arrow Price/Stock"
 F 12 "C8678" H 5500 4250 50  0001 C CNN "LCSC"
+F 13 "SS34B-HF" H 5500 4250 50  0001 C CNN "MPN"
+F 14 "0.0350" H 5500 4250 50  0001 C CNN "Price"
+F 15 "0" H 5500 4250 50  0001 C CNN "source"
 	1    5500 4250
 	0    1    1    0
@@
 F 4 "Schottky Diodes & Rectifiers DIODE SCHOTTKY 3A 40V SMB" H 6125 2425 50  0001 L CNN "Description"
 F 5 "3.2" H 6125 2325 50  0001 L CNN "Height"
-F 6 "Comchip Technology" H 6125 2225 50  0001 L CNN "Manufacturer_Name"
-F 7 "SS34B-HF" H 6125 2125 50  0001 L CNN "Manufacturer_Part_Number"
+F 6 "" H 6125 2225 50  0001 L CNN "Manufacturer_Name"
+F 7 "" H 6125 2125 50  0001 L CNN "Manufacturer_Part_Number"
 F 8 "750-SS34B-HF" H 6125 2025 50  0001 L CNN "Mouser Part Number"
 F 9 "https://www.mouser.co.uk/ProductDetail/Comchip-Technology/SS34B-HF/?qs=vmHwEFxEFR9G1M%252BcUPG%2FxQ%3D%3D" H 6125 1925 50  0001 L CNN "Mouser Price/Stock"
@@
 F 11 "" H 6125 1725 50  0001 L CNN "Arrow Price/Stock"
 F 12 "C8678" H 5625 2475 50  0001 C CNN "LCSC"
+F 13 "SS34B-HF" H 5625 2475 50  0001 C CNN "MPN"
+F 14 "0.0350" H 5625 2475 50  0001 C CNN "Price"
+F 15 "0" H 5625 2475 50  0001 C CNN "source"
 	1    5625 2475
 	0    1    1    0

Commit message: minor updates
Parts:
- C2, C33: Price (none) -> 0.0549
Changed lines of the file:
@@
 F 5 "CL31A106KBHNNNE" H 2825 2750 50  0001 C CNN "MPN"
 F 6 "0" H 2825 2750 50  0001 C CNN "source"
+F 7 "0.0549" H 2825 2750 50  0001 C CNN "Price"
 	1    2825 2750
 	1    0    0    -1
@@
 F 5 "CL31A106KBHNNNE" H 2800 4525 50  0001 C CNN "MPN"
 F 6 "0" H 2800 4525 50  0001 C CNN "source"
+F 7 "0.0549" H 2800 4525 50  0001 C CNN "Price"
 	1    2800 4525
 	1    0    0    -1

Commit message: ENC28j60 package changed to soic 28 17.9
TODO: route
Parts:
- J2: LCSC (none) -> N/A
Changed lines of the file:
@@
 F 3 "~" H 2325 1475 50  0001 C CNN
 F 4 "Connector unknown" H 2325 1475 50  0001 C CNN "Mpn"
+F 5 "N/A" H 2325 1475 50  0001 C CNN "LCSC"
 	1    2325 1475
 	-1   0    0    1
