File: small/analog_in.sch (KiCad schematic (older format))
At the start: 20 parts, among them U1 LM358

Commit message: BOM updated
Layout changed
Parts:
- C22, C23: MPN (none) -> CL21B102KBCNNNC; source (none) -> 0
- C6, FB1, FB2, U1: source (none) -> 0
- D32, D38: MPN (none) -> P6SMB30CA; Price (none) -> 0.0756; source (none) -> 1
- D34, D35, D39, D40: source (none) -> 1
- R25, R26: MPN (none) -> 0603WAF1001T5E; source (none) -> 0
- R32, R33: MPN (none) -> 0805W8F3601T5E; source (none) -> 0
- R35, R37: MPN (none) -> 0805W8F5600T5E; source (none) -> 0
Changed lines of the file:
@@
 F 5 "BAT54S L44" H 3025 2000 50  0001 C CNN "MPN"
 F 6 "0.0178" H 3025 2000 50  0001 C CNN "Price"
+F 7 "1" H 3025 2000 50  0001 C CNN "source"
 	1    3025 2000
 	1    0    0    -1
@@
 F 3 "https://datasheet.lcsc.com/szlcsc/Littelfuse-P6SMB30A_C80390.pdf" H 1550 2350 50  0001 C CNN
 F 4 "C320521" V 1600 2350 50  0001 C CNN "LCSC"
+F 5 "P6SMB30CA" H 1600 2350 50  0001 C CNN "MPN"
+F 6 "0.0756" H 1600 2350 50  0001 C CNN "Price"
+F 7 "1" H 1600 2350 50  0001 C CNN "source"
 	1    1600 2350
 	0    1    1    0
@@
 F 4 "C46653" H 3025 2450 50  0001 C CNN "LCSC"
 F 5 "0.0127" H 3025 2450 50  0001 C CNN "Price"
+F 6 "CL21B102KBCNNNC" H 3025 2450 50  0001 C CNN "MPN"
+F 7 "0" H 3025 2450 50  0001 C CNN "source"
 	1    3025 2450
 	1    0    0    -1
@@
 F 4 "C46653" H 3075 4475 50  0001 C CNN "LCSC"
 F 5 "0.0127" H 3075 4475 50  0001 C CNN "Price"
+F 6 "CL21B102KBCNNNC" H 3075 4475 50  0001 C CNN "MPN"
+F 7 "0" H 3075 4475 50  0001 C CNN "source"
 	1    3075 4475
 	1    0    0    -1
@@
 F 4 "0.0035" V 1875 2200 50  0001 C CNN "Price"
 F 5 "C18359" V 1875 2200 50  0001 C CNN "LCSC"
+F 6 "0805W8F3601T5E" H 1875 2200 50  0001 C CNN "MPN"
+F 7 "0" H 1875 2200 50  0001 C CNN "source"
 	1    1875 2200
 	0    -1   -1   0
@@
 F 4 "0.0044" V 2250 2400 50  0001 C CNN "Price"
 F 5 "C28636" V 2250 2400 50  0001 C CNN "LCSC"
+F 6 "0805W8F5600T5E" H 2250 2400 50  0001 C CNN "MPN"
+F 7 "0" H 2250 2400 50  0001 C CNN "source"
 	1    2250 2400
 	-1   0    0    1
@@
 F 6 "BAT54S L44" H 3075 4025 50  0001 C CNN "Mpn"
 F 7 "0.0178" H 3075 4025 50  0001 C CNN "Price"
+F 8 "1" H 3075 4025 50  0001 C CNN "source"
 	1    3075 4025
 	1    0    0    -1
@@
 F 5 "BAT54S L44" H 5445 4125 50  0001 C CNN "MPN"
 F 6 "0.0178" H 5445 4125 50  0001 C CNN "Price"
+F 7 "1" H 5445 4125 50  0001 C CNN "source"
 	1    5445 4125
 	1    0    0    -1
@@
 F 3 "https://datasheet.lcsc.com/szlcsc/Littelfuse-P6SMB30A_C80390.pdf" H 1625 4375 50  0001 C CNN
 F 4 "C320521" V 1675 4375 50  0001 C CNN "LCSC"
+F 5 "P6SMB30CA" H 1675 4375 50  0001 C CNN "MPN"
+F 6 "0.0756" H 1675 4375 50  0001 C CNN "Price"
+F 7 "1" H 1675 4375 50  0001 C CNN "source"
 	1    1675 4375
 	0    1    1    0
@@
 F 4 "0.0035" V 1950 4225 50  0001 C CNN "Price"
 F 5 "C18359" V 1950 4225 50  0001 C CNN "LCSC"
+F 6 "0805W8F3601T5E" H 1950 4225 50  0001 C CNN "MPN"
+F 7 "0" H 1950 4225 50  0001 C CNN "source"
 	1    1950 4225
 	0    -1   -1   0
@@
 F 5 "LM358DR2G" H 4200 4325 50  0001 C CNN "MPN"
 F 6 "0.0687" H 4200 4325 50  0001 C CNN "Price"
+F 7 "0" H 4200 4325 50  0001 C CNN "source"
 	2    4200 4325
 	1    0    0    -1
@@
 F 5 "GZ2012D601TF" V 2650 2200 50  0001 C CNN "MPN"
 F 6 "0.0121" V 2650 2200 50  0001 C CNN "Price"
+F 7 "0" H 2650 2200 50  0001 C CNN "source"
 	1    2650 2200
 	0    1    1    0
@@
 F 5 "GZ2012D601TF" V 2725 4225 50  0001 C CNN "MPN"
 F 6 "0.0121" V 2725 4225 50  0001 C CNN "Price"
+F 7 "0" H 2725 4225 50  0001 C CNN "source"
 	1    2725 4225
 	0    1    1    0
@@
 F 5 "0.0071" H 2275 6025 50  0001 C CNN "Price"
 F 6 "CC0603KRX7R9BB104" H 2275 6025 50  0001 C CNN "MPN"
+F 7 "0" H 2275 6025 50  0001 C CNN "source"
 	1    2275 6025
 	1    0    0    -1
@@
 F 6 "BAT54S L44" H 5295 2100 50  0001 C CNN "Mpn"
 F 7 "0.0178" H 5295 2100 50  0001 C CNN "Price"
+F 8 "1" H 5295 2100 50  0001 C CNN "source"
 	1    5295 2100
 	1    0    0    -1
@@
 F 4 " C21190" H 4900 2300 50  0001 C CNN "LCSC"
 F 5 "0.009" H 4900 2300 50  0001 C CNN "Price"
+F 6 "0603WAF1001T5E" H 4900 2300 50  0001 C CNN "MPN"
+F 7 "0" H 4900 2300 50  0001 C CNN "source"
 	1    4900 2300
 	0    1    1    0
@@
 F 4 " C21190" H 4925 4325 50  0001 C CNN "LCSC"
 F 5 "0.009" H 4925 4325 50  0001 C CNN "Price"
+F 6 "0603WAF1001T5E" H 4925 4325 50  0001 C CNN "MPN"
+F 7 "0" H 4925 4325 50  0001 C CNN "source"
 	1    4925 4325
 	0    1    1    0
@@
 F 4 "0.0044" V 2325 4425 50  0001 C CNN "Price"
 F 5 "C28636" V 2325 4425 50  0001 C CNN "LCSC"
+F 6 "0805W8F5600T5E" H 2325 4425 50  0001 C CNN "MPN"
+F 7 "0" H 2325 4425 50  0001 C CNN "source"
 	1    2325 4425
 	-1   0    0    1

Commit message: ENC28j60 package changed to soic 28 17.9
TODO: route
Parts:
- R25, R26: LCSC C21190 -> C21190
- R34, R36: LCSC na -> N/A; Price na -> N/A
- U1: LCSC (none) -> N/A
Changed lines of the file:
@@
 F 1 "na" V 2400 2050 50  0000 C CNN
 F 2 "Resistor_SMD:R_0603_1608Metric" V 2180 2050 50  0001 C CNN
-F 3 "na" H 2250 2050 50  0001 C CNN
-F 4 "na" V 2250 2050 50  0001 C CNN "Price"
-F 5 "na" V 2250 2050 50  0001 C CNN "LCSC"
+F 3 "N/A" H 2250 2050 50  0001 C CNN
+F 4 "N/A" V 2250 2050 50  0001 C CNN "Price"
+F 5 "N/A" V 2250 2050 50  0001 C CNN "LCSC"
 	1    2250 2050
 	-1   0    0    1
@@
 F 1 "na" V 2475 4075 50  0000 C CNN
 F 2 "Resistor_SMD:R_0603_1608Metric" V 2255 4075 50  0001 C CNN
-F 3 "na" H 2325 4075 50  0001 C CNN
-F 4 "na" V 2325 4075 50  0001 C CNN "Price"
-F 5 "na" V 2325 4075 50  0001 C CNN "LCSC"
+F 3 "N/A" H 2325 4075 50  0001 C CNN
+F 4 "N/A" V 2325 4075 50  0001 C CNN "Price"
+F 5 "N/A" V 2325 4075 50  0001 C CNN "LCSC"
 	1    2325 4075
 	-1   0    0    1
@@
 F 2 "Package_SO:SOIC-8_3.9x4.9mm_P1.27mm" H 4175 2300 50  0001 C CNN
 F 3 "http://www.ti.com/lit/ds/symlink/lm2904-n.pdf" H 4175 2300 50  0001 C CNN
+F 4 "N/A" H 4175 2300 50  0001 C CNN "LCSC"
 	1    4175 2300
 	1    0    0    -1
@@
 F 2 "Package_SO:SOIC-8_3.9x4.9mm_P1.27mm" H 1650 6050 50  0001 C CNN
 F 3 "http://www.ti.com/lit/ds/symlink/lm2904-n.pdf" H 1650 6050 50  0001 C CNN
+F 4 "N/A" H 1650 6050 50  0001 C CNN "LCSC"
 	3    1650 6050
 	1    0    0    -1
@@
 F 2 "Resistor_SMD:R_0603_1608Metric" V 4830 2300 50  0001 C CNN
 F 3 "https://eu.mouser.com/datasheet/2/427/crcwce3-1762584.pdf" H 4900 2300 50  0001 C CNN
-F 4 " C21190" H 4900 2300 50  0001 C CNN "LCSC"
+F 4 "C21190" H 4900 2300 50  0001 C CNN "LCSC"
 F 5 "0.009" H 4900 2300 50  0001 C CNN "Price"
 F 6 "0603WAF1001T5E" H 4900 2300 50  0001 C CNN "MPN"
@@
 F 2 "Resistor_SMD:R_0603_1608Metric" V 4855 4325 50  0001 C CNN
 F 3 "https://eu.mouser.com/datasheet/2/427/crcwce3-1762584.pdf" H 4925 4325 50  0001 C CNN
-F 4 " C21190" H 4925 4325 50  0001 C CNN "LCSC"
+F 4 "C21190" H 4925 4325 50  0001 C CNN "LCSC"
 F 5 "0.009" H 4925 4325 50  0001 C CNN "Price"
 F 6 "0603WAF1001T5E" H 4925 4325 50  0001 C CNN "MPN"

Commit message: working on JLCPCB orientations
Parts:
- U1: LCSC N/A -> C7950
Changed lines of the file:
@@
 F 2 "Package_SO:SOIC-8_3.9x4.9mm_P1.27mm" H 4175 2300 50  0001 C CNN
 F 3 "http://www.ti.com/lit/ds/symlink/lm2904-n.pdf" H 4175 2300 50  0001 C CNN
-F 4 "N/A" H 4175 2300 50  0001 C CNN "LCSC"
+F 4 "C7950" H 4175 2300 50  0001 C CNN "LCSC"
 	1    4175 2300
 	1    0    0    -1
