File: small/digital_input.sch (KiCad schematic (older format))
At the start: 12 parts, among them U6 EL357N(C)(TA)-G, U7 EL357N(C)(TA)-G

Commit message: GPS connector moved,
antenna matching networks removed

SUPERCAPACITOR from jlpcb used.
Parts:
- U6, U7: LCSC (none) -> C29981; LCSC# C29981 -> (none)
Changed lines of the file:
@@
 F 4 "$0.0520" H 3375 1925 50  0001 C CNN "CMPN"
 F 5 "EL357N(C)(TA)-G" H 3375 1925 50  0001 C CNN "MPN"
-F 6 "C29981" H 3375 1925 50  0001 C CNN "LCSC#"
+F 6 "" H 3375 1925 50  0001 C CNN "LCSC#"
+F 7 "C29981" H 3375 1925 50  0001 C CNN "LCSC"
 	1    3375 1925
 	1    0    0    -1
@@
 F 4 "$0.0520" H 3400 3750 50  0001 C CNN "CMPN"
 F 5 "EL357N(C)(TA)-G" H 3400 3750 50  0001 C CNN "MPN"
-F 6 "C29981" H 3400 3750 50  0001 C CNN "LCSC#"
+F 6 "" H 3400 3750 50  0001 C CNN "LCSC#"
+F 7 "C29981" H 3400 3750 50  0001 C CNN "LCSC"
 	1    3400 3750
 	1    0    0    -1

Commit message: BOM updated
Layout changed
Parts:
- C12, C13: MPN (none) -> CL21B102KBCNNNC; source (none) -> 0
- D1, D2: MPN (none) -> P6SMB30CA; source (none) -> 1
- D5, D6: source (none) -> 1
- R10: MPN (none) -> 0805W8F5101T5E; source (none) -> 0
- R13, R14: MPN (none) -> 0805W8F1001T5E; Price 0.0756 -> 0.0040; source (none) -> 0
- R9: LCSC C27834 -> C27834; MPN (none) -> 0805W8F5101T5E; source (none) -> 0
- U6, U7: source (none) -> 0
Changed lines of the file:
@@
 F 6 "BAT54S L44" H 2525 1375 50  0001 C CNN "Mpn"
 F 7 "0.0178" H 2525 1375 50  0001 C CNN "Price"
+F 8 "1" H 2525 1375 50  0001 C CNN "source"
 	1    2525 1375
 	1    0    0    -1
@@
 F 4 "C46653" H 2525 2075 50  0001 C CNN "LCSC"
 F 5 "0.0127" H 2525 2075 50  0001 C CNN "Price"
+F 6 "CL21B102KBCNNNC" H 2525 2075 50  0001 C CNN "MPN"
+F 7 "0" H 2525 2075 50  0001 C CNN "source"
 	1    2525 2075
 	1    0    0    -1
@@
 F 6 "" H 3375 1925 50  0001 C CNN "LCSC#"
 F 7 "C29981" H 3375 1925 50  0001 C CNN "LCSC"
+F 8 "0" H 3375 1925 50  0001 C CNN "source"
 	1    3375 1925
 	1    0    0    -1
@@
 F 2 "Resistor_SMD:R_0805_2012Metric" V 1905 1825 50  0001 C CNN
 F 3 "https://datasheet.lcsc.com/szlcsc/Uniroyal-Elec-0805W8F5101T5E_C27834.pdf" H 1975 1825 50  0001 C CNN
-F 4 " C27834" V 1975 1825 50  0001 C CNN "LCSC"
+F 4 "C27834" V 1975 1825 50  0001 C CNN "LCSC"
 F 5 "0.0039" V 1975 1825 50  0001 C CNN "Price"
+F 6 "0805W8F5101T5E" H 1975 1825 50  0001 C CNN "MPN"
+F 7 "0" H 1975 1825 50  0001 C CNN "source"
 	1    1975 1825
 	0    1    1    0
@@
 F 3 "https://datasheet.lcsc.com/szlcsc/Uniroyal-Elec-0805W8F1001T5E_C17513.pdf" H 3675 1300 50  0001 C CNN
 F 4 "C17513" V 3675 1300 50  0001 C CNN "LCSC"
-F 5 "0.0756" V 3675 1300 50  0001 C CNN "Price"
+F 5 "0.0040" V 3675 1300 50  0001 C CNN "Price"
+F 6 "0805W8F1001T5E" H 3675 1300 50  0001 C CNN "MPN"
+F 7 "0" H 3675 1300 50  0001 C CNN "source"
 	1    3675 1300
 	-1   0    0    1
@@
 F 4 "C27834" V 2000 3650 50  0001 C CNN "LCSC"
 F 5 "0.0039" V 2000 3650 50  0001 C CNN "Price"
+F 6 "0805W8F5101T5E" H 2000 3650 50  0001 C CNN "MPN"
+F 7 "0" H 2000 3650 50  0001 C CNN "source"
 	1    2000 3650
 	0    1    1    0
@@
 F 6 "" H 3400 3750 50  0001 C CNN "LCSC#"
 F 7 "C29981" H 3400 3750 50  0001 C CNN "LCSC"
+F 8 "0" H 3400 3750 50  0001 C CNN "source"
 	1    3400 3750
 	1    0    0    -1
@@
 F 4 "C46653" H 2550 3900 50  0001 C CNN "LCSC"
 F 5 "0.0127" H 2550 3900 50  0001 C CNN "Price"
+F 6 "CL21B102KBCNNNC" H 2550 3900 50  0001 C CNN "MPN"
+F 7 "0" H 2550 3900 50  0001 C CNN "source"
 	1    2550 3900
 	1    0    0    -1
@@
 F 4 "C320521" V 1250 3800 50  0001 C CNN "LCSC"
 F 5 "0.0756" V 1250 3800 50  0001 C CNN "Price"
+F 6 "P6SMB30CA" H 1250 3800 50  0001 C CNN "MPN"
+F 7 "1" H 1250 3800 50  0001 C CNN "source"
 	1    1250 3800
 	0    1    1    0
@@
 F 6 "BAT54S L44" H 2550 3200 50  0001 C CNN "Mpn"
 F 7 "0.0178" H 2550 3200 50  0001 C CNN "Price"
+F 8 "1" H 2550 3200 50  0001 C CNN "source"
 	1    2550 3200
 	1    0    0    -1
@@
 F 3 "https://datasheet.lcsc.com/szlcsc/Uniroyal-Elec-0805W8F1001T5E_C17513.pdf" H 3700 3125 50  0001 C CNN
 F 4 "C17513" V 3700 3125 50  0001 C CNN "LCSC"
-F 5 "0.0756" V 3700 3125 50  0001 C CNN "Price"
+F 5 "0.0040" V 3700 3125 50  0001 C CNN "Price"
+F 6 "0805W8F1001T5E" H 3700 3125 50  0001 C CNN "MPN"
+F 7 "0" H 3700 3125 50  0001 C CNN "source"
 	1    3700 3125
 	-1   0    0    1
@@
 F 4 "C320521" V 1225 1975 50  0001 C CNN "LCSC"
 F 5 "0.0756" V 1225 1975 50  0001 C CNN "Price"
+F 6 "P6SMB30CA" H 1225 1975 50  0001 C CNN "MPN"
+F 7 "1" H 1225 1975 50  0001 C CNN "source"
 	1    1225 1975
 	0    1    1    0

Commit message: minor updates
Parts:
- U6, U7: Price (none) -> 0.0850
Changed lines of the file:
@@
 F 7 "C29981" H 3375 1925 50  0001 C CNN "LCSC"
 F 8 "0" H 3375 1925 50  0001 C CNN "source"
+F 9 "0.0850" H 3375 1925 50  0001 C CNN "Price"
 	1    3375 1925
 	1    0    0    -1
@@
 F 7 "C29981" H 3400 3750 50  0001 C CNN "LCSC"
 F 8 "0" H 3400 3750 50  0001 C CNN "source"
+F 9 "0.0850" H 3400 3750 50  0001 C CNN "Price"
 	1    3400 3750
 	1    0    0    -1

Commit message: iso voltage update
minor changes
Parts:
- R10: value 5k -> 2.2k; LCSC C27834 -> C17520; MPN 0805W8F5101T5E -> 0805W8F2201T5E; Price 0.0039 -> 0.0042
- R9: value 5k -> 2.2k; LCSC C27834 -> C17520; MPN 0805W8F5101T5E -> 0805W8F2201T5E
Changed lines of the file:
@@
 AR Path="/652E8962/65324E52" Ref="R9"  Part="1"
 F 0 "R9" V 1768 1825 50  0000 C CNN
-F 1 "5k" V 1859 1825 50  0000 C CNN
+F 1 "2.2k" V 1859 1825 50  0000 C CNN
 F 2 "Resistor_SMD:R_0805_2012Metric" V 1905 1825 50  0001 C CNN
-F 3 "https://datasheet.lcsc.com/szlcsc/Uniroyal-Elec-0805W8F5101T5E_C27834.pdf" H 1975 1825 50  0001 C CNN
-F 4 "C27834" V 1975 1825 50  0001 C CNN "LCSC"
+F 3 "https://datasheet.lcsc.com/szlcsc/Uniroyal-Elec-0805W8F2201T5E_C17520.pdf" H 1975 1825 50  0001 C CNN
+F 4 "C17520" V 1975 1825 50  0001 C CNN "LCSC"
 F 5 "0.0039" V 1975 1825 50  0001 C CNN "Price"
-F 6 "0805W8F5101T5E" H 1975 1825 50  0001 C CNN "MPN"
+F 6 "0805W8F2201T5E" H 1975 1825 50  0001 C CNN "MPN"
 F 7 "0" H 1975 1825 50  0001 C CNN "source"
 	1    1975 1825
@@
 AR Path="/652E8962/65324EC9" Ref="R10"  Part="1"
 F 0 "R10" V 1793 3650 50  0000 C CNN
-F 1 "5k" V 1884 3650 50  0000 C CNN
+F 1 "2.2k" V 1884 3650 50  0000 C CNN
 F 2 "Resistor_SMD:R_0805_2012Metric" V 1930 3650 50  0001 C CNN
-F 3 "https://datasheet.lcsc.com/szlcsc/Uniroyal-Elec-0805W8F5101T5E_C27834.pdf" H 2000 3650 50  0001 C CNN
-F 4 "C27834" V 2000 3650 50  0001 C CNN "LCSC"
-F 5 "0.0039" V 2000 3650 50  0001 C CNN "Price"
-F 6 "0805W8F5101T5E" H 2000 3650 50  0001 C CNN "MPN"
+F 3 "https://datasheet.lcsc.com/szlcsc/Uniroyal-Elec-0805W8F2201T5E_C17520.pdf" H 2000 3650 50  0001 C CNN
+F 4 "C17520" V 2000 3650 50  0001 C CNN "LCSC"
+F 5 "0.0042" V 2000 3650 50  0001 C CNN "Price"
+F 6 "0805W8F2201T5E" H 2000 3650 50  0001 C CNN "MPN"
 F 7 "0" H 2000 3650 50  0001 C CNN "source"
 	1    2000 3650
